File: board/semaphore.kicad_sch (KiCad schematic)
At the start: 13 parts, among them J1 BAT, J2 D1x, J3 D2x, Q1 2N3904, Q2 2N3904

Commit message: WIP
Parts:
- added R5, R6: 10k, Resistor_THT:R_Axial_DIN0207_L6.3mm_D2.5mm_P10.16mm_Horizontal, symbol Device:R
- added U1: ATtiny412-SS, Package_SO:SOIC-8_3.9x4.9mm_P1.27mm, symbol MCU_Microchip_ATtiny:ATtiny412-SS
Connections:
- net BAT+: now also R5.1, R6.1; no longer J1.2 (Pin_2)
- net BAT-: no longer J1.1 (Pin_1)
- net D2-: now also R6.2
- net at C1.2, Q1.2 (B): now also R5.2
Other:
- moved on the sheet: J1, R2, R3
